File: esp-expander.kicad_pcb (KiCad board)
At the start: 2 copper layers, 56 parts, among them J1 Programming Header, J2 HR911105A, Q1 AO3401A, SW1 RESET, U1 ESP32-WROOM-32D, U2 AMS1117-3.3, U3 MCP23017_SS, U4 LAN8720A

Commit message: Added lcsc part nums
Parts:
- added J3: Conn_01x16, Connector_PinHeader_2.54mm:PinHeader_1x16_P2.54mm_Vertical, F.Cu at (105.2, 94.6)
- added J4: Conn_01x16, Connector_PinHeader_2.54mm:PinHeader_1x16_P2.54mm_Vertical, F.Cu at (109.9, 94.6)
- C1, C2, C9: value 100nF/6.3V -> 100nF/50V/10%
- C10, C11, C15, C16, C6, C7: value 100nF -> 100nF/50V/10%
- C12: value 470pF -> 470pF/50V/20%
- C13, C17: value 1uF -> 1uF/10%/25V
- C14: value 4.7uF -> 4.7uF/10V/20%
- C3: value 22uF/6.3V -> 22uF/6.3V/20%
- C4: value 100uF/16V -> 100uF/10V/20%; footprint Capacitor_SMD:CP_Elec_4x5.4 -> Capacitor_SMD:CP_Elec_5x5.4
- C5, C8: value 10uF -> 10uF/6.3V/20%
- D1: value LED -> LED Red; footprint LED_SMD:LED_0402_1005Metric -> LED_SMD:LED_0603_1608Metric
- F1: value Fuse -> 6V 500mA 100A
- L1: value L -> PZ1608D121-2R0TF
- R1: value 2K2 -> 1K/1/16W/50V
- R2: value 10K -> 10K/1/16W/50V
- R20, R21: value 1K -> 1K/1/16W/50V
- R3, R4: value 4K7 -> 4K7/1/16W/50V
- R5, R6: value 100K -> 100K/1/16W/50V
- SW1: footprint Button_Switch_SMD:SW_SPST_B3U-1000P -> Button_Switch_SMD:SW_SPST_EVPBF
