File: esp-expander.kicad_pcb (KiCad board)
At the start: 2 copper layers, 58 parts, among them J1 Programming Header, J2 HR911105A, J3 Conn_01x16, J4 Conn_01x16, Q1 AO3401A, SW1 RESET, U1 ESP32-WROOM-32D, U2 AMS1117-3.3, U3 MCP23017_SS, U4 LAN8720A

Commit message: Added schematic
Parts:
- added JP2: 3.3VJumper, Jumper:SolderJumper-2_P1.3mm_Open_Pad1.0x1.5mm, F.Cu at (179.8, 131.4)
- J3: footprint Connector_PinHeader_2.54mm:PinHeader_1x16_P2.54mm_Vertical -> Connector_PinHeader_2.54mm:PinHeader_1x18_P2.54mm_Vertical; moved to B.Cu
- J4: value Conn_01x16 -> Conn_01x12; footprint Connector_PinHeader_2.54mm:PinHeader_1x16_P2.54mm_Vertical -> Connector_PinHeader_2.54mm:PinHeader_1x12_P2.54mm_Vertical; moved to B.Cu
- moved J2 62.1 mm to (104.2, 71.8), turned to 270 degrees
- moved U1 39.3 mm to (98.2, 98.7), turned to 180 degrees
- moved J3 34.6 mm to (82.9, 68.1), turned to 180 degrees
- moved R5 27.1 mm to (173.9, 141.7)
- moved Q1 21.4 mm to (173.9, 138.3), turned to 90 degrees
- moved U2 18.6 mm to (180.2, 136.5)
- moved C5 17.8 mm to (177.0, 141.7)
- moved C6 16.9 mm to (177.0, 140.7)
- moved R6 16.7 mm to (173.9, 140.6), turned to 180 degrees
- moved F1 15.3 mm to (173.9, 135.5), turned to 180 degrees
- moved C8 14.1 mm to (177.5, 131.2), turned to 180 degrees
- moved J4 11.9 mm to (113.9, 83.4), turned to 180 degrees
- moved JP1 8.92 mm to (191.0, 97.5)
- moved C7 8.17 mm to (177.5, 132.3), turned to 180 degrees
- moved C9 7.98 mm to (199.6, 85.5), turned to 270 degrees
Connections:
- F1 pad 2: (no net) -> VCC
- J3 pad 1: (no net) -> +3V3
- J3 pad 10: (no net) -> /MCP/MCP9
- J3 pad 11: (no net) -> /MCP/MCP10
- J3 pad 12: (no net) -> /MCP/MCP11
- J3 pad 13: (no net) -> /MCP/MCP12
- J3 pad 14: (no net) -> /MCP/MCP13
- J3 pad 15: (no net) -> /MCP/MCP14
- J3 pad 16: (no net) -> /MCP/MCP15
- J3 pad 2: (no net) -> /MCP/MCP1
- J3 pad 3: (no net) -> /MCP/MCP2
- J3 pad 4: (no net) -> /MCP/MCP3
- J3 pad 5: (no net) -> /MCP/MCP4
- J3 pad 6: (no net) -> /MCP/MCP5
- J3 pad 7: (no net) -> /MCP/MCP6
- J3 pad 8: (no net) -> /MCP/MCP7
- J3 pad 9: (no net) -> /MCP/MCP8
- J4 pad 1: (no net) -> VCC
- J4 pad 10: (no net) -> PROGRAMMING_GPIO0
- J4 pad 11: (no net) -> PROGRAMMING_TX
- J4 pad 12: (no net) -> PROGRAMMING_RX
- J4 pad 2: (no net) -> GND
- J4 pad 3: (no net) -> +3V3
- J4 pad 4: (no net) -> DIGITAL1
- J4 pad 5: (no net) -> DIGITAL2
- J4 pad 6: (no net) -> DIGITAL3
- J4 pad 7: (no net) -> DIGITAL4
- J4 pad 8: (no net) -> DIGITAL5
- J4 pad 9: (no net) -> PROGRAMMING_RESET
- U1 pad 26: (no net) -> DIGITAL1
- U1 pad 27: (no net) -> DIGITAL2
- U1 pad 29: (no net) -> DIGITAL3
- U1 pad 8: (no net) -> DIGITAL4
- U1 pad 9: (no net) -> DIGITAL5
- U3 pad 1: (no net) -> /MCP/MCP9
- U3 pad 2: (no net) -> /MCP/MCP10
- U3 pad 21: (no net) -> /MCP/MCP1
- U3 pad 22: (no net) -> /MCP/MCP2
- U3 pad 23: (no net) -> /MCP/MCP3
- U3 pad 24: (no net) -> /MCP/MCP4
- U3 pad 25: (no net) -> /MCP/MCP5
- U3 pad 26: (no net) -> /MCP/MCP6
- U3 pad 27: (no net) -> /MCP/MCP7
- U3 pad 28: (no net) -> /MCP/MCP8
- U3 pad 3: (no net) -> /MCP/MCP11
- U3 pad 4: (no net) -> /MCP/MCP12
- U3 pad 5: (no net) -> /MCP/MCP13
- U3 pad 6: (no net) -> /MCP/MCP14
- U3 pad 7: (no net) -> /MCP/MCP15
- U3 pad 8: (no net) -> /MCP/MCP16

Commit message: Basic layout done
Parts:
- moved J1 111.0 mm to (82.6, 106.0), turned to 90 degrees
- moved C9 110.1 mm to (89.5, 82.3), turned to 0 degrees
- moved JP1 109.2 mm to (82.7, 111.1), turned to 90 degrees
- moved U3 107.5 mm to (87.0, 87.6), turned to 90 degrees
- moved C5 94.5 mm to (100.1, 86.8), turned to 270 degrees
- moved R5 93.9 mm to (100.1, 83.7), turned to 270 degrees
- moved C12 93.8 mm to (82.3, 68.1), turned to 180 degrees
- moved C6 93.0 mm to (101.1, 86.8), turned to 270 degrees
- moved C14 92.6 mm to (82.3, 65.9), turned to 180 degrees
- moved R6 92.3 mm to (101.2, 83.7), turned to 90 degrees
- moved C13 90.8 mm to (82.3, 67.0), turned to 180 degrees
- moved C11 90.1 mm to (82.3, 72.4)
- moved Q1 89.0 mm to (103.5, 83.7), turned to 0 degrees
- moved C10 88.3 mm to (82.3, 71.3)
- moved U2 88.1 mm to (105.3, 90.0), turned to 270 degrees
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Other:
- board outline added: 37.6 x 56.9 mm
