File: power.sch (KiCad schematic (older format))
At the start: 9 parts

Commit message: Exported first net
Parts:
- gave numbers to parts that had none: 9
Changed lines of the file:
@@
 $EndDescr
 $Comp
-L power:VCC #PWR?
+L power:VCC #PWR0112
 U 1 1 6213E359
 P 4150 3250
-F 0 "#PWR?" H 4150 3100 50  0001 C CNN
+F 0 "#PWR0112" H 4150 3100 50  0001 C CNN
 F 1 "VCC" V 4165 3377 50  0000 L CNN
 F 2 "" H 4150 3250 50  0001 C CNN
@@
 $EndComp
 $Comp
-L Regulator_Linear:AMS1117-3.3 U?
+L Regulator_Linear:AMS1117-3.3 U2
 U 1 1 6213EB1B
 P 6100 3250
-F 0 "U?" H 6100 3492 50  0000 C CNN
+F 0 "U2" H 6100 3492 50  0000 C CNN
 F 1 "AMS1117-3.3" H 6100 3401 50  0000 C CNN
 F 2 "Package_TO_SOT_SMD:SOT-223-3_TabPin2" H 6100 3450 50  0001 C CNN
@@
 P 5700 3450
 AR Path="/6212150F/6213FDEB" Ref="C?"  Part="1"
-AR Path="/6213DFD4/6213FDEB" Ref="C?"  Part="1"
-F 0 "C?" H 5600 3550 50  0000 L CNN
+AR Path="/6213DFD4/6213FDEB" Ref="C6"  Part="1"
+F 0 "C6" H 5600 3550 50  0000 L CNN
 F 1 "100nF" V 5850 3350 50  0000 L CNN
 F 2 "Capacitor_SMD:C_0402_1005Metric" H 5738 3300 50  0001 C CNN
@@
 P 5400 3450
 AR Path="/6212150F/6213FE5D" Ref="C?"  Part="1"
-AR Path="/6213DFD4/6213FE5D" Ref="C?"  Part="1"
-F 0 "C?" H 5300 3550 50  0000 L CNN
+AR Path="/6213DFD4/6213FE5D" Ref="C5"  Part="1"
+F 0 "C5" H 5300 3550 50  0000 L CNN
 F 1 "10uF" V 5550 3350 50  0000 L CNN
 F 2 "Capacitor_SMD:C_0402_1005Metric" H 5438 3300 50  0001 C CNN
@@
 P 6450 3450
 AR Path="/6212150F/62140191" Ref="C?"  Part="1"
-AR Path="/6213DFD4/62140191" Ref="C?"  Part="1"
-F 0 "C?" H 6350 3550 50  0000 L CNN
+AR Path="/6213DFD4/62140191" Ref="C7"  Part="1"
+F 0 "C7" H 6350 3550 50  0000 L CNN
 F 1 "100nF" V 6600 3350 50  0000 L CNN
 F 2 "Capacitor_SMD:C_0402_1005Metric" H 6488 3300 50  0001 C CNN
@@
 P 6750 3450
 AR Path="/6212150F/621406EF" Ref="C?"  Part="1"
-AR Path="/6213DFD4/621406EF" Ref="C?"  Part="1"
-F 0 "C?" H 6650 3550 50  0000 L CNN
+AR Path="/6213DFD4/621406EF" Ref="C8"  Part="1"
+F 0 "C8" H 6650 3550 50  0000 L CNN
 F 1 "10uF" V 6900 3350 50  0000 L CNN
 F 2 "Capacitor_SMD:C_0402_1005Metric" H 6788 3300 50  0001 C CNN
@@
 $EndComp
 $Comp
-L power:GND #PWR?
+L power:GND #PWR0113
 U 1 1 62144941
 P 5400 3650
-F 0 "#PWR?" H 5400 3400 50  0001 C CNN
+F 0 "#PWR0113" H 5400 3400 50  0001 C CNN
 F 1 "GND" H 5405 3477 50  0000 C CNN
 F 2 "" H 5400 3650 50  0001 C CNN
@@
 $EndComp
 $Comp
-L power:GND #PWR?
+L power:GND #PWR0114
 U 1 1 62144C75
 P 5700 3650
-F 0 "#PWR?" H 5700 3400 50  0001 C CNN
+F 0 "#PWR0114" H 5700 3400 50  0001 C CNN
 F 1 "GND" H 5705 3477 50  0000 C CNN
 F 2 "" H 5700 3650 50  0001 C CNN
@@
 $EndComp
 $Comp
-L power:GND #PWR?
+L power:GND #PWR0115
 U 1 1 62144E93
 P 6100 3650
-F 0 "#PWR?" H 6100 3400 50  0001 C CNN
+F 0 "#PWR0115" H 6100 3400 50  0001 C CNN
 F 1 "GND" H 6105 3477 50  0000 C CNN
 F 2 "" H 6100 3650 50  0001 C CNN
@@
 $EndComp
 $Comp
-L power:GND #PWR?
+L power:GND #PWR0116
 U 1 1 62145207
 P 6450 3650
-F 0 "#PWR?" H 6450 3400 50  0001 C CNN
+F 0 "#PWR0116" H 6450 3400 50  0001 C CNN
 F 1 "GND" H 6455 3477 50  0000 C CNN
 F 2 "" H 6450 3650 50  0001 C CNN
@@
 $EndComp
 $Comp
-L power:GND #PWR?
+L power:GND #PWR0117
 U 1 1 62145604
 P 6750 3650
-F 0 "#PWR?" H 6750 3400 50  0001 C CNN
+F 0 "#PWR0117" H 6750 3400 50  0001 C CNN
 F 1 "GND" H 6755 3477 50  0000 C CNN
 F 2 "" H 6750 3650 50  0001 C CNN
@@
 	6750 3600 6750 3650
 $Comp
-L power:+3.3V #PWR?
+L power:+3.3V #PWR0118
 U 1 1 621461FB
 P 6750 3200
-F 0 "#PWR?" H 6750 3050 50  0001 C CNN
+F 0 "#PWR0118" H 6750 3050 50  0001 C CNN
 F 1 "+3.3V" H 6765 3373 50  0000 C CNN
 F 2 "" H 6750 3200 50  0001 C CNN
@@
 	5700 3250 5800 3250
 $Comp
-L Transistor_FET:AO3401A Q?
+L Transistor_FET:AO3401A Q1
 U 1 1 62147B60
 P 4750 3350
-F 0 "Q?" V 5092 3350 50  0000 C CNN
+F 0 "Q1" V 5092 3350 50  0000 C CNN
 F 1 "AO3401A" V 5001 3350 50  0000 C CNN
 F 2 "Package_TO_SOT_SMD:SOT-23" H 4950 3275 50  0001 L CIN
@@
 $EndComp
 $Comp
-L power:GND #PWR?
+L power:GND #PWR0119
 U 1 1 621497A9
 P 4750 4050
-F 0 "#PWR?" H 4750 3800 50  0001 C CNN
+F 0 "#PWR0119" H 4750 3800 50  0001 C CNN
 F 1 "GND" H 4755 3877 50  0000 C CNN
 F 2 "" H 4750 4050 50  0001 C CNN
@@
 $EndComp
 $Comp
-L Device:R R?
+L Device:R R6
 U 1 1 6214A951
 P 5000 3450
-F 0 "R?" H 5070 3496 50  0000 L CNN
+F 0 "R6" H 5070 3496 50  0000 L CNN
 F 1 "100K" H 5070 3405 50  0000 L CNN
 F 2 "Resistor_SMD:R_0402_1005Metric" V 4930 3450 50  0001 C CNN
@@
 $EndComp
 $Comp
-L Device:R R?
+L Device:R R5
 U 1 1 6214B479
 P 4750 3850
-F 0 "R?" H 4820 3896 50  0000 L CNN
+F 0 "R5" H 4820 3896 50  0000 L CNN
 F 1 "100K" H 4820 3805 50  0000 L CNN
 F 2 "Resistor_SMD:R_0402_1005Metric" V 4680 3850 50  0001 C CNN
@@
 Connection ~ 5400 3250
 $Comp
-L Device:Fuse F?
+L Device:Fuse F1
 U 1 1 62151104
 P 4350 3250
-F 0 "F?" V 4153 3250 50  0000 C CNN
+F 0 "F1" V 4153 3250 50  0000 C CNN
 F 1 "Fuse" V 4244 3250 50  0000 C CNN
 F 2 "Fuse:Fuse_0805_2012Metric" V 4280 3250 50  0001 C CNN

Commit message: Added lcsc part nums
Parts:
- C5, C8: value 10uF -> 10uF/6.3V/20%; LCSC (none) -> C15525
- C6, C7: value 100nF -> 100nF/50V/10%; LCSC (none) -> C307331
- F1: value Fuse -> 6V 500mA 100A; LCSC (none) -> C135329
- Q1: LCSC (none) -> C15127
- R5, R6: value 100K -> 100K/1/16W/50V; LCSC (none) -> C25741
- U2: LCSC (none) -> C6186
Other:
- moved on the sheet: C5, C6, C7, C8, F1, Q1, R5, R6, U2

Commit message: Added schematic
Parts:
- added JP2: 3.3VJumper, Jumper:SolderJumper-2_P1.3mm_Open_Pad1.0x1.5mm, symbol Device:Jumper_NO_Small
Connections:
- net +3V3: now also JP2.2
- net at C5.1, C6.1, Q1.2 (S)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: now also JP2.1
Changed lines of the file:
@@
 Wire Wire Line
 	4150 3500 4200 3500
+$Comp
+L Device:Jumper_NO_Small JP2
+U 1 1 6225CAF5
+P 6100 3150
+F 0 "JP2" H 6100 3335 50  0000 C CNN
+F 1 "3.3VJumper" H 6100 3244 50  0000 C CNN
+F 2 "Jumper:SolderJumper-2_P1.3mm_Open_Pad1.0x1.5mm" H 6100 3150 50  0001 C CNN
+F 3 "~" H 6100 3150 50  0001 C CNN
+	1    6100 3150
+	1    0    0    -1
+$EndComp
+Wire Wire Line
+	5700 3500 5700 3150
+Wire Wire Line
+	5700 3150 6000 3150
+Wire Wire Line
+	6450 3500 6450 3150
+Wire Wire Line
+	6450 3150 6200 3150
 $EndSCHEMATC
